Commit message: transmission work

File: ur5/ur_with_gripper.xacro (robot description, xacro)
@@ -274,4 +274,41 @@
         </actuator>
     </transmission>
+    <transmission name="robotiq_85_left_knuckle_trans">
+        <type>transmission_interface/SimpleTransmission</type>
+        <joint name="robotiq_85_left_knuckle_joint">
+            <hardwareInterface>hardware_interface/PositionJointInterface</hardwareInterface>
+        </joint>
+        <actuator name="robotiq_85_left_knuckle_motor">
+            <mechanicalReduction>1</mechanicalReduction>
+            <hardwareInterface>hardware_interface/PositionJointInterface</hardwareInterface>
+        </actuator>
+    </transmission>
+    <!-- Mimic joints -->
+    <gazebo>
+        <plugin filename="libgazebo_mimic_joint_plugin.so" name="mimic_robotiq_85_1">
+            <joint>robotiq_85_left_knuckle_joint</joint>
+            <mimicJoint>robotiq_85_right_knuckle_joint</mimicJoint>
+        </plugin>
+        <plugin filename="libgazebo_mimic_joint_plugin.so" name="mimic_robotiq_85_2">
+            <joint>robotiq_85_left_knuckle_joint</joint>
+            <mimicJoint>robotiq_85_left_inner_knuckle_joint</mimicJoint>
+        </plugin>
+        <plugin filename="libgazebo_mimic_joint_plugin.so" name="mimic_robotiq_85_3">
+            <joint>robotiq_85_left_knuckle_joint</joint>
+            <mimicJoint>robotiq_85_right_inner_knuckle_joint</mimicJoint>
+        </plugin>
+        <plugin filename="libgazebo_mimic_joint_plugin.so" name="mimic_robotiq_85_4">
+            <joint>robotiq_85_left_knuckle_joint</joint>
+            <mimicJoint>robotiq_85_left_finger_tip_joint</mimicJoint>
+            <multiplier>-1.0</multiplier>
+            <offset>0.0</offset>
+        </plugin>
+        <plugin filename="libgazebo_mimic_joint_plugin.so" name="mimic_robotiq_85_5">
+            <joint>robotiq_85_left_knuckle_joint</joint>
+            <mimicJoint>robotiq_85_right_finger_tip_joint</mimicJoint>
+            <multiplier>-1.0</multiplier>
+            <offset>0.0</offset>
+        </plugin>
+    </gazebo>
     <!-- nothing to do here at the moment -->
     <joint name="robotiq_85_base_joint" type="fixed">
